Commit message: Fix ur10 robot with the three grippers.

File: urdf/robot.xacro (robot description, xacro)
@@ -2,18 +2,42 @@
 <robot xmlns:xacro="http://www.ros.org/wiki/xacro"
        name="ur10" >
-  <xacro:property name="include_gripper" value="$(arg include_gripper)"/>
+  <xacro:arg name="tipo_gripper" default="jaco"/>
+  <xacro:property name="p_gripper_name" value="$(arg tipo_gripper)"/>
   <!-- ur10 -->
   <xacro:include filename="$(find manipulacion_pkg)/urdf/ur10_macro.xacro" />
-  <xacro:if value="$(arg include_gripper)">
+  <!-- When using schunk hand-->
+  <xacro:if value="${p_gripper_name == 'schunk'}">
+    <xacro:include filename="$(find manipulacion_pkg)/urdf/schunk_hand.xacro"/>
+    <xacro:schunk_hand schunk_prefix="hand" parent="tool0"  mass_divider="1" finger_mass_divider="1"
+                    activate_gravity="$(arg activate_gravity)" floating_gripper="$(arg floating_gripper)">
+      <origin xyz="0.0 0 0" rpy="0 -1.5708 0"/>
+    </xacro:schunk_hand>
+  </xacro:if>
+  <xacro:if value="${p_gripper_name == 'robotiq'}">
+    <xacro:include filename="$(find manipulacion_pkg)/urdf/robotiq_hand.xacro"/>
+    <xacro:robotiq_3f_hand prefix="hand" parent="tool0"  mass_divider="1" finger_mass_divider="1"
+                    activate_gravity="$(arg activate_gravity)" floating_gripper="$(arg floating_gripper)">
+      <origin xyz="0.0 0 0" rpy="0 0 1.5708"/>
+    </xacro:robotiq_3f_hand>
+  </xacro:if>
+  <!-- When using jaco_hand -->
+  <xacro:if value="${p_gripper_name == 'jaco'}">
     <xacro:include filename="$(find manipulacion_pkg)/urdf/jaco_hand.xacro" />
+    <xacro:jaco_hand jaco_prefix="hand" parent="tool0"  mass_divider="1" finger_mass_divider="1"
+                    activate_gravity="$(arg activate_gravity)" floating_gripper="$(arg floating_gripper)">
+      <origin xyz="0 0 0" rpy=" 0 0 0"/>
+    </xacro:jaco_hand>
   </xacro:if>
+  <!-- <xacro:if value="$(arg include_gripper)">
+    <xacro:include filename="$(find manipulacion_pkg)/urdf/jaco_hand.xacro" />
+  </xacro:if> -->
   <!-- arm -->
   <xacro:ur10_robot prefix="" transmission_hw_interface="hardware_interface/EffortJointInterface"/>
   <!-- gripper -->
-  <xacro:if value="$(arg include_gripper)">
+  <!-- <xacro:if value="$(arg include_gripper)">
     <xacro:jaco_hand jaco_prefix="hand" parent="tool0"  mass_divider="5" finger_mass_divider="5" activate_gravity="false" floating_gripper="false">
       <origin xyz="-0.01 0 0" rpy="1.57 0 0"/>
     </xacro:jaco_hand>
-  </xacro:if>
+  </xacro:if> -->
   <!-- world will be root link-->
   <link name="world" />

File: urdf/ur10_macro.xacro (robot description, xacro)
@@ -19,8 +19,8 @@
   <xacro:macro name="ur10_robot" params="
    prefix
-   joint_limits_parameters_file:='$(find ur_description)/config/ur10/joint_limits.yaml'
-   kinematics_parameters_file:='$(find ur_description)/config/ur10/default_kinematics.yaml'
-   physical_parameters_file:='$(find ur_description)/config/ur10/physical_parameters.yaml'
-   visual_parameters_file:='$(find ur_description)/config/ur10/visual_parameters.yaml'
+   joint_limits_parameters_file:='$(find manipulacion_pkg)/config/ur10/joint_limits.yaml'
+   kinematics_parameters_file:='$(find manipulacion_pkg)/config/ur10/default_kinematics.yaml'
+   physical_parameters_file:='$(find manipulacion_pkg)/config/ur10/physical_parameters.yaml'
+   visual_parameters_file:='$(find manipulacion_pkg)/config/ur10/visual_parameters.yaml'
    transmission_hw_interface:=hardware_interface/PositionJointInterface
    safety_limits:=false

File: urdf/ur_macro.xacro (robot description, xacro)
@@ -42,6 +42,6 @@
      - Muhammad Asif Rana
   -->
-  <xacro:include filename="$(find ur_description)/urdf/inc/ur_transmissions.xacro" />
-  <xacro:include filename="$(find ur_description)/urdf/inc/ur_common.xacro" />
+  <xacro:include filename="$(find manipulacion_pkg)/urdf/ur_transmissions.xacro" />
+  <xacro:include filename="$(find manipulacion_pkg)/urdf/ur_common.xacro" />
   <xacro:macro name="ur_robot" params="
     prefix
@@ -64,5 +64,6 @@
     <xacro:ur_arm_transmission prefix="${prefix}" hw_interface="${transmission_hw_interface}" />
     <!-- links: main serial chain -->
-    <link name="${prefix}base_link">
+    <link name="${prefix}base_link"/>
+    <!-- <link name="${prefix}base_link">
       <visual>
         <origin xyz="0 0 0.15" rpy="0 0 0"/>
@@ -77,5 +78,5 @@
         </geometry>
       </collision>
-    </link>
+    </link> -->
     <link name="${prefix}base_link_inertia">
       <visual>
@@ -239,5 +240,5 @@
          <safety_controller soft_lower_limit="${shoulder_pan_lower_limit + safety_pos_margin}" soft_upper_limit="${shoulder_pan_upper_limit - safety_pos_margin}" k_position="${safety_k_position}" k_velocity="0.0"/>
       </xacro:if>
-      <dynamics damping="0" friction="0"/>
+      <dynamics damping="0.1" friction="0.1"/>
     </joint>
     <joint name="${prefix}shoulder_lift_joint" type="revolute">
@@ -251,5 +252,5 @@
          <safety_controller soft_lower_limit="${shoulder_lift_lower_limit + safety_pos_margin}" soft_upper_limit="${shoulder_lift_upper_limit - safety_pos_margin}" k_position="${safety_k_position}" k_velocity="0.0"/>
       </xacro:if>
-      <dynamics damping="0" friction="0"/>
+      <dynamics damping="0.1" friction="0.1"/>
     </joint>
     <joint name="${prefix}elbow_joint" type="revolute">
@@ -263,5 +264,5 @@
          <safety_controller soft_lower_limit="${elbow_joint_lower_limit + safety_pos_margin}" soft_upper_limit="${elbow_joint_upper_limit - safety_pos_margin}" k_position="${safety_k_position}" k_velocity="0.0"/>
       </xacro:if>
-      <dynamics damping="0" friction="0"/>
+      <dynamics damping="0.1" friction="0.1"/>
     </joint>
     <joint name="${prefix}wrist_1_joint" type="revolute">
@@ -275,5 +276,5 @@
          <safety_controller soft_lower_limit="${wrist_1_lower_limit + safety_pos_margin}" soft_upper_limit="${wrist_1_upper_limit - safety_pos_margin}" k_position="${safety_k_position}" k_velocity="0.0"/>
       </xacro:if>
-      <dynamics damping="0" friction="0"/>
+      <dynamics damping="0.1" friction="0.1"/>
     </joint>
     <joint name="${prefix}wrist_2_joint" type="revolute">
@@ -287,5 +288,5 @@
          <safety_controller soft_lower_limit="${wrist_2_lower_limit + safety_pos_margin}" soft_upper_limit="${wrist_2_upper_limit - safety_pos_margin}" k_position="${safety_k_position}" k_velocity="0.0"/>
       </xacro:if>
-      <dynamics damping="0" friction="0"/>
+      <dynamics damping="0.1" friction="0.1"/>
     </joint>
     <joint name="${prefix}wrist_3_joint" type="revolute">
@@ -299,5 +300,5 @@
          <safety_controller soft_lower_limit="${wrist_3_lower_limit + safety_pos_margin}" soft_upper_limit="${wrist_3_upper_limit - safety_pos_margin}" k_position="${safety_k_position}" k_velocity="0.0"/>
       </xacro:if>
-      <dynamics damping="0" friction="0"/>
+      <dynamics damping="0.1" friction="0.1"/>
     </joint>
     <link name="${prefix}base"/>
