Commit message: Fix collisionDetection.

File: urdf/jaco.urdf (robot description, URDF)
Before this commit: robot caja_simple_robot, 2 links, 1 joints
Links:
- link link_caja: geometry collision box size=0.21 0.2 0.1; visual box size=0.21 0.2 0.1
Joints:
- joint base_to_caja_joint: origin xyz=-0.0 0 0 rpy=0 0 0 -> xyz=0.0 0 0 rpy=0 0 0
